Commit message: Add the description of the robot in the urdf file

File: my_rb1_description/urdf/my_rb1_robot.urdf (robot description, URDF)
Before this commit: robot my_robot, 7 links, 6 joints
Links:
- link back_caster: mass 0.5 -> 6.25
- link front_caster: mass 0.5 -> 6.25
- link front_laser: geometry collision cylinder length=0.15 radius=0.025; visual cylinder length=0.05 radius=0.025
- link left_wheel: mass 1 -> 12.5
- link right_wheel: mass 1 -> 12.5
Joints:
- joint base_to_back_caster: origin xyz=0.1 0 0 -> xyz=-0.1 0 0
- joint base_to_front_caster: origin xyz=-0.1 0 0 -> xyz=0.1 0 0
- joint base_to_front_laser: axis 1 0 0 -> 0 0 1
- joint base_to_left_wheel: origin xyz=0 -0.2 0 -> xyz=0 0.2 0
- joint base_to_right_wheel: origin xyz=0 0.2 0 -> xyz=0 -0.2 0

Commit message: Creation of a package my_rb1_gazebo and related modification to make the robot in gazebo

File: my_rb1_description/urdf/my_rb1_robot.urdf (robot description, URDF)
Before this commit: robot my_robot, 7 links, 6 joints
Joints:
- joint base_footprint_to_base_link: child base_link -> base_footprint; parent base_footprint -> base_link
- joint base_to_back_caster: origin xyz=-0.1 0 0 -> xyz=-0.1 0 -0.15
- joint base_to_front_caster: origin xyz=0.1 0 0 -> xyz=0.1 0 -0.15
- joint base_to_front_laser: type continuous -> fixed
- joint base_to_left_wheel: origin xyz=0 0.2 0 -> xyz=0 0.2 -0.15
- joint base_to_right_wheel: origin xyz=0 -0.2 0 -> xyz=0 -0.2 -0.15

Commit message: Add the modification for the task3

File: my_rb1_description/urdf/my_rb1_robot.urdf (robot description, URDF)
Before this commit: robot my_robot, 7 links, 6 joints
Joints:
- joint base_footprint_to_base_link: origin xyz=0 0 0 -> xyz=0 0 -0.15
- joint base_to_back_caster: type continuous -> fixed
- joint base_to_front_caster: type continuous -> fixed

Commit message: Add the correction needed for reevaluation

File: my_rb1_description/urdf/my_rb1_robot.urdf (robot description, URDF)
Before this commit: robot my_robot, 7 links, 6 joints
Joints:
- joint base_to_front_laser: axis 0 0 1 -> (none); origin xyz=0.25 0 0.075 -> xyz=0.25 0 0.075 rpy=3.14 0 0
- joint base_to_left_wheel: axis 0 1 0 -> 0 -1 0; child left_wheel -> right_wheel; origin xyz=0 0.2 -0.15 -> xyz=0 -0.2 -0.15
- joint base_to_right_wheel: axis 0 1 0 -> 0 -1 0; child right_wheel -> left_wheel; origin xyz=0 -0.2 -0.15 -> xyz=0 0.2 -0.15
